Commit message: created_core_urdf

File: description/robot.urdf.xacro (robot description, xacro)
@@ -1,4 +1,110 @@
 <?xml version="1.0"?>
 <robot xmlns:xacro="http://www.ros.org/wiki/xacro"  name="robot">
-    <xacro:include filename="robot_core.xacro"/>
+    <xacro:include filename="inertial_macros.xacro"/>
+    <!-- <material name="white">
+        <color rgba="1 1 1 1 ">
+    </material>
+    <material name="orange">
+        <color rgba="1 0.3 0.1 1">
+    </material>
+    <material name="blue">
+        <color rgba="0.2 0.2 1 1">
+    </material>
+    <material name="black">
+        <color rgba="0 0 0 1">
+    </material> -->
+    <!-- base link  -->
+    <link name="base_link">
+    </link>
+    <!-- chassis link  -->
+    <joint name ="chassis_joint" type="fixed">
+        <parent link="base_link"/>
+        <child link="chassis"/>
+        <origin xyz="-0.1 0 0"/>
+    </joint>
+    <link name="chassis">
+        <visual>
+            <origin xyz="0.15 0 0.075"/>
+            <geometry>
+                <box size="0.3 0.3 0.15 "/>
+            </geometry>
+        </visual>
+        <collision>
+            <origin xyz="0.15 0 0.075"/>
+            <geometry>
+                <box size="0.3 0.3 0.15 "/>
+            </geometry>
+        </collision>
+        <xacro:inertial_box mass="0.5" x="0.3" y ="0.3" z="0.15">
+            <origin xyz="0.15 0 0.075" rpy="0 0 0"/>
+        </xacro:inertial_box>
+    </link>
+        <!-- left wheel joint  -->
+    <joint name= "left_wheel_joint" type="continuous">
+        <parent link="base_link"/>
+        <child link="left_wheel"/>
+        <origin xyz="0 0.175 0" rpy="-${pi/2} 0 0"/>
+        <axis xyz="0 0 1"/>
+    </joint>
+    <link name="left_wheel">
+        <visual>
+            <geometry>
+                <cylinder radius="0.05" length ="0.04"/>
+            </geometry>
+            <!-- <material name="blue"/> -->
+        </visual>
+        <collision>
+            <geometry>
+                <cylinder radius="0.05" length ="0.04"/>
+            </geometry>
+        </collision>
+        <xacro:inertial_cylinder mass="0.1" length="0.04" radius="0.050">
+            <origin xyz="0 0 0" rpy="0 0 0" />
+        </xacro:inertial_cylinder>
+    </link>
+      <!-- right wheel joint  -->
+    <joint name= "right_wheel_joint" type="continuous">
+        <parent link="base_link"/>
+        <child link="right_wheel"/>
+        <origin xyz="0 -0.175 0" rpy="${pi/2} 0 0"/>
+        <axis xyz="0 0 -1"/>
+    </joint>
+    <link name="right_wheel">
+        <visual>
+            <geometry>
+                <cylinder radius="0.05" length ="0.04"/>
+            </geometry>
+            <!-- <material name="blue"/> -->
+        </visual>
+        <collision>
+            <geometry>
+                <cylinder radius="0.05" length ="0.04"/>
+            </geometry>
+        </collision>
+        <xacro:inertial_cylinder mass="0.1" length="0.04" radius="0.050">
+            <origin xyz="0 0 0" rpy="0 0 0" />
+        </xacro:inertial_cylinder>
+    </link>
+    <!-- carster wheel link  -->
+    <joint name="caster_wheel_joint" type="fixed">
+        <parent link="chassis"/>
+        <child link="caster_wheel"/>
+        <origin xyz="0.24 0 0"/>
+    </joint>
+    <link name="caster_wheel">
+        <visual>
+            <geometry>
+                <sphere radius="0.05"/>
+                <!-- <material name="black"/> -->
+            </geometry>
+        </visual>
+        <collision>
+            <geometry>
+                <sphere radius="0.05"/>
+            </geometry>
+        </collision>
+        <xacro:inertial_sphere mass="0.1" radius="0.05">
+            <origin xyz="0 0 0" rpy ="0 0 0"/>
+        </xacro:inertial_sphere>
+    </link>
 </robot>

Commit message: created_gazebo_file

File: description/robot.urdf.xacro (robot description, xacro)
@@ -2,4 +2,5 @@
 <robot xmlns:xacro="http://www.ros.org/wiki/xacro"  name="robot">
     <xacro:include filename="inertial_macros.xacro"/>
+    <xacro:include filename="gazebo_control.xacro"/>
     <!-- <material name="white">
         <color rgba="1 1 1 1 ">
@@ -40,4 +41,7 @@
         </xacro:inertial_box>
     </link>
+    <gazebo reference="chassis">
+        <!-- <material>Gazebo/Black</material> -->
+    </gazebo>
         <!-- left wheel joint  -->
     <joint name= "left_wheel_joint" type="continuous">
@@ -63,4 +67,7 @@
         </xacro:inertial_cylinder>
     </link>
+    <gazebo reference="left_wheel">
+        <!-- <material>Gazebo/Black</material> -->
+    </gazebo>
       <!-- right wheel joint  -->
     <joint name= "right_wheel_joint" type="continuous">
@@ -86,4 +93,7 @@
         </xacro:inertial_cylinder>
     </link>
+    <gazebo reference="right_wheel">
+        <!-- <material>Gazebo/Black</material> -->
+    </gazebo>
     <!-- carster wheel link  -->
     <joint name="caster_wheel_joint" type="fixed">
@@ -108,3 +118,24 @@
         </xacro:inertial_sphere>
     </link>
+    <gazebo reference="caster_wheel">
+        <!-- <material>Gazebo/Black</material> -->
+    </gazebo>
+    <gazebo>
+        <plugin name="diff_drive" filename="libgazebo_ros_diff_drive.so">
+        <!-- Wheel Information -->
+        <left_joint>left_wheel_joint</left_joint>
+        <right_joint>right_wheel_joint</right_joint>
+        <wheel_separation>0.35</wheel_separation>
+        <wheel_diameter>0.1</wheel_diameter>
+        <!-- Limits -->
+        <max_wheel_torque>200</max_wheel_torque>
+        <max_wheel_acceleration>10.0</max_wheel_acceleration>
+        <!-- Output -->
+        <odometry_frame>odom</odometry_frame>
+        <robot_base_frame>base_link</robot_base_frame>
+        <publish_odom>true</publish_odom>
+        <publish_odom_tf>true</publish_odom_tf>
+        <publish_wheel_tf>true</publish_wheel_tf>
+        </plugin>
+    </gazebo>
 </robot>
